File: arte/preamp/preamp.sch (KiCad schematic (older format))
At the start: 22 parts, among them U1 AD8643, U10 AD8643, U11 AD8643, U12 AD8643, U13 AD8643, U14 AD8643, U15 AD8643, U16 AD8643, U2 AD8643, U3 AD8643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

Commit message: First version of kikad eib and preamp files
Parts:
- added BackLED2, FrontLED2: LED, symbol LED
- added R3, R4: 1 kOhm, symbol R
Connections:
- net VCC: no longer BackLED1.1 (A), FrontLED1.1 (A)
- net VDD: no longer R1.2, R2.2
- net LED_VCC: now reaches Output-Conn1.2 (PIN2)
- net LED_VCC: now also BackLED1.1 (A), FrontLED1.1 (A), BackLED2.1 (A), FrontLED2.1 (A)
- net LED_VDD: now reaches Output-Conn1.36 (PIN36)
- net LED_VDD: now also R1.2, R2.2, R3.2, R4.2
- new net: BackLED2.2 (K), R4.1
- new net: FrontLED2.2 (K), R3.1
Other:
- moved on the sheet: BackLED1, FrontLED1, R1, R2
Changed lines of the file:
@@
-EESchema Schematic File Version 2  date Mon 24 Feb 2014 07:32:48 PM EST
+EESchema Schematic File Version 2  date Thu 13 Mar 2014 03:55:04 PM EDT
 LIBS:power
 LIBS:device
@@
 Sheet 1 1
 Title ""
-Date "24 feb 2014"
+Date "13 mar 2014"
 Rev ""
 Comp ""
@@
 Comment4 ""
 $EndDescr
-Wire Wire Line
-	11000 2250 11000 900
+Text Label 10900 5650 0    60   ~ 0
+LED_VDD
+Text Label 9400 2350 0    60   ~ 0
+LED_VCC
+Text Label 11000 1600 0    60   ~ 0
+LED_VDD
+Text Label 9300 1600 0    60   ~ 0
+LED_VCC
+Wire Wire Line
+	9300 1600 9300 650
+Wire Wire Line
+	11000 1600 11000 650
+Connection ~ 11000 1300
+Wire Wire Line
+	10850 1300 11000 1300
+Connection ~ 11000 850
+Wire Wire Line
+	10850 850  11000 850
+Wire Wire Line
+	10250 850  10350 850
+Wire Wire Line
+	10250 1300 10350 1300
 Wire Wire Line
 	3250 650  3350 650
@@
 Wire Wire Line
 	3950 1000 3950 1100
-Wire Wire Line
-	11000 2250 10900 2250
-Connection ~ 11000 1350
-Wire Wire Line
-	10850 1350 11000 1350
-Wire Wire Line
-	10250 1350 10350 1350
-Connection ~ 9300 1350
-Wire Wire Line
-	9850 1350 9300 1350
+Connection ~ 11000 1100
+Wire Wire Line
+	10850 1100 11000 1100
+Wire Wire Line
+	10250 1100 10350 1100
+Connection ~ 9300 1100
+Wire Wire Line
+	9850 1100 9300 1100
 Wire Notes Line
 	9100 1450 9100 6950
@@
 	2600 1200 2600 6900
 Wire Wire Line
-	9400 2250 9300 2250
-Wire Wire Line
-	9300 2250 9300 900
-Wire Wire Line
-	9300 900  9850 900
-Wire Wire Line
-	10250 900  10350 900
-Wire Wire Line
-	11000 900  10850 900
+	9300 650  9850 650
+Wire Wire Line
+	10250 650  10350 650
+Wire Wire Line
+	11000 650  10850 650
 Wire Wire Line
 	3950 1250 3950 1350
@@
 Wire Wire Line
 	6150 650  6250 650
+Wire Wire Line
+	9850 850  9300 850
+Connection ~ 9300 850
+Wire Wire Line
+	9850 1300 9300 1300
+Connection ~ 9300 1300
+$Comp
+L LED FrontLED2
+U 1 1 530BEC27
+P 10050 850
+F 0 "FrontLED2" H 9700 900 50  0000 C CNN
+F 1 "LED" H 10050 750 50  0000 C CNN
+	1    10050 850
+	1    0    0    -1
+$EndComp
+$Comp
+L LED BackLED2
+U 1 1 530BEC26
+P 10050 1300
+F 0 "BackLED2" H 9700 1350 50  0000 C CNN
+F 1 "LED" H 10050 1200 50  0000 C CNN
+	1    10050 1300
+	1    0    0    -1
+$EndComp
+$Comp
+L R R3
+U 1 1 530BEC25
+P 10600 850
+F 0 "R3" V 10680 850 50  0000 C CNN
+F 1 "1 kOhm" V 10600 850 50  0000 C CNN
+	1    10600 850
+	0    -1   -1   0
+$EndComp
+$Comp
+L R R4
+U 1 1 530BEC24
+P 10600 1300
+F 0 "R4" V 10680 1300 50  0000 C CNN
+F 1 "1 kOhm" V 10600 1300 50  0000 C CNN
+	1    10600 1300
+	0    -1   -1   0
+$EndComp
 Text Label 5750 6800 0    60   ~ 0
 P45
@@
 L R R2
 U 1 1 53062D9A
-P 10600 1350
-F 0 "R2" V 10680 1350 50  0000 C CNN
-F 1 "1 kOhm" V 10600 1350 50  0000 C CNN
-	1    10600 1350
+P 10600 1100
+F 0 "R2" V 10680 1100 50  0000 C CNN
+F 1 "1 kOhm" V 10600 1100 50  0000 C CNN
+	1    10600 1100
 	0    -1   -1   0
 $EndComp
@@
 L R R1
 U 1 1 53062D91
-P 10600 900
-F 0 "R1" V 10680 900 50  0000 C CNN
-F 1 "1 kOhm" V 10600 900 50  0000 C CNN
-	1    10600 900
+P 10600 650
+F 0 "R1" V 10680 650 50  0000 C CNN
+F 1 "1 kOhm" V 10600 650 50  0000 C CNN
+	1    10600 650
 	0    -1   -1   0
 $EndComp
@@
 L LED BackLED1
 U 1 1 53062D8B
-P 10050 1350
-F 0 "BackLED1" H 10050 1450 50  0000 C CNN
-F 1 "LED" H 10050 1250 50  0000 C CNN
-	1    10050 1350
+P 10050 1100
+F 0 "BackLED1" H 9700 1150 50  0000 C CNN
+F 1 "LED" H 10050 1000 50  0000 C CNN
+	1    10050 1100
 	1    0    0    -1
 $EndComp
@@
 L LED FrontLED1
 U 1 1 53062D82
-P 10050 900
-F 0 "FrontLED1" H 10050 1000 50  0000 C CNN
-F 1 "LED" H 10050 800 50  0000 C CNN
-	1    10050 900
-	1    0    0    -1
-$EndComp
+P 10050 650
+F 0 "FrontLED1" H 9700 700 50  0000 C CNN
+F 1 "LED" H 10050 550 50  0000 C CNN
+	1    10050 650
+	1    0    0    -1
+$EndComp
