File: arte-hardware/eib/eib.sch (KiCad schematic (older format))
At the start: 44 parts

Commit message: add svg prints of schematics for eib and preamp
Other:
- note added: "EIB V4 ImAlsoGreg@gmail.com sciencetypes.com"
Changed lines of the file:
@@
-EESchema Schematic File Version 2  date Wed 19 Feb 2014 12:56:00 PM EST
+EESchema Schematic File Version 2  date Wed 26 Mar 2014 05:11:30 PM EDT
 LIBS:power
 LIBS:device
@@
 Sheet 1 1
 Title ""
-Date "17 feb 2014"
+Date "26 mar 2014"
 Rev ""
 Comp ""
@@
 Comment4 ""
 $EndDescr
+Text Notes 1000 7400 0    60   ~ 0
+EIB V4    ImAlsoGreg@gmail.com    sciencetypes.com
 Wire Wire Line
 	4800 7150 4900 7150
