File: arte-hardware/preamp/preamp.sch (KiCad schematic (older format))
At the start: 26 parts, among them U1 AD8643, U10 AD8643, U11 AD8643, U12 AD8643, U13 AD8643, U14 AD8643, U15 AD8643, U16 AD8643, U2 AD8643, U3 AD8643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

Commit message: add svg prints of schematics for eib and preamp
Other:
- note added: "Preamp"
- note added: "V4\n"
- note added: "imalsogreg@gmail.com sciencetypes.com"
Changed lines of the file:
@@
-EESchema Schematic File Version 2  date Thu 13 Mar 2014 03:55:04 PM EDT
+EESchema Schematic File Version 2  date Wed 26 Mar 2014 05:14:57 PM EDT
 LIBS:power
 LIBS:device
@@
 Sheet 1 1
 Title ""
-Date "13 mar 2014"
+Date "26 mar 2014"
 Rev ""
 Comp ""
@@
 Comment4 ""
 $EndDescr
+Text Notes 8600 7400 0    60   ~ 0
+imalsogreg@gmail.com    sciencetypes.com
+Text Notes 10700 7700 0    60   ~ 0
+V4\n
+Text Notes 8050 7550 0    60   ~ 0
+Preamp
 Text Label 10900 5650 0    60   ~ 0
 LED_VDD

Commit message: version 5 preamp - small vias, pads at board edge
Other:
- note added: "V5\n"
- note removed: "V4\n"
Changed lines of the file:
@@
-EESchema Schematic File Version 2  date Wed 26 Mar 2014 05:14:57 PM EDT
+EESchema Schematic File Version 2  date Thu 03 Apr 2014 02:00:47 PM EDT
 LIBS:power
 LIBS:device
@@
 Sheet 1 1
 Title ""
-Date "26 mar 2014"
+Date "3 apr 2014"
 Rev ""
 Comp ""
@@
 imalsogreg@gmail.com    sciencetypes.com
 Text Notes 10700 7700 0    60   ~ 0
-V4\n
+V5\n
 Text Notes 8050 7550 0    60   ~ 0
 Preamp
