File: arte-hardware/16-tet-patchbox/patchboxfinal.kicad_pcb (KiCad board)
At the start: 2 copper layers, 54 parts

Commit message: updated board and fixed a bug in power circuit and ground islands
Parts:
- NegR1, dropoutR1: value (none) -> GS3
Connections:
- D2 pad 1: GND -> N-000043
- NegR1 pad 1: N-000043 -> GND
- NegR1 pad 2: GND -> N-000043
Routing:
- net GND: track 1613.9 -> 1512.5 mm
- net /a: track 808.7 -> 837.2 mm
- net N-000043: track 14.7 -> 35.5 mm, vias 0 -> 1
- net /-5: track 194.7 -> 177.4 mm, vias 1 -> 3
- net /s9: track 83.4 -> 96.7 mm
- net N-000057: track 226.3 -> 237.6 mm, vias 2 -> 4
- net N-000054: track 32.9 -> 22.3 mm
- net /+5: track 116.4 -> 125.2 mm
- net /s16: track 85.6 -> 90.3 mm
- net /LED+5: track 148.1 -> 152.6 mm
- net N-000053: track 18.2 -> 14.5 mm
- net /12d: track 200.5 -> 203.7 mm
- net /13c: track 192.4 -> 195.6 mm
- net /13d: track 209.2 -> 212.3 mm
- net /11a: track 215.5 -> 212.6 mm
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Other:
- board outline added: 391.7 x 179.3 mm
- board text added: "+"
- board text added: "-"
- board text added: "16 Tetrode Patchbox v1.0 Hannah Wirtshafter hsw@mit.edu"
- board text added: "S10"
- board text added: "S9"
